File: _autosave-power_stage.kicad_sch (KiCad schematic)
At the start: 27 parts, among them J1 Input, J1 Output, Q1 IMW120R014M1H, Q2 IMW120R014M1H, Q6 2N7002BK,215, U4 TC4432VOA

Commit message: updated the design
Changed lines of the file:
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@@
     (stroke (width 0) (type default))
+  )
+  (circle (center 236.22 97.79) (radius 28.6525)
+    (stroke (width 0) (type default))
+    (fill (type none))
+  )
+  (circle (center 124.46 77.47) (radius 9.1581)
+    (stroke (width 0) (type default))
+    (fill (type none))
   )
   (global_label "VSOURCE" (shape input) (at 190.5 85.09 180) (fields_autoplaced)
