File: Current sense Amplifier.kicad_sch (KiCad schematic)
At the start: 18 parts, among them U2 MCP6022

Commit message: updated the design
Parts:
- added TP9 (x2): 5001, 5001 tp:KEYSTONE_5001, symbol 5001:5001
Connections:
- net I_SENSE_ANB4: now also TP9.TP
- net I_SENSE_C3IN1-: now also TP9.TP
Changed lines of the file:
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@@
+    (stroke (width 0) (type default))
+  )
+  (wire (pts (xy 187.96 68.58) (xy 187.96 73.66))
     (stroke (width 0) (type default))
   )
@@
   )
   (wire (pts (xy 191.77 110.49) (xy 201.93 110.49))
+    (stroke (width 0) (type default))
+  )
+  (wire (pts (xy 191.77 105.41) (xy 191.77 110.49))
     (stroke (width 0) (type default))
   )
@@
     )
   )
+  (symbol (lib_id "5001:5001") (at 187.96 63.5 90) (unit 1)
+    (in_bom yes) (on_board yes) (dnp no) (fields_autoplaced)
+    (property "Reference" "TP9" (at 190.5 62.23 90)
+      (effects (font (size 1.27 1.27)) (justify right))
+    )
+    (property "Value" "5001" (at 190.5 64.77 90)
+      (effects (font (size 1.27 1.27)) (justify right))
+    )
+    (property "Footprint" "5001 tp:KEYSTONE_5001" (at 187.96 63.5 0)
+      (effects (font (size 1.27 1.27)) (justify bottom) hide)
+    )
+    (property "Datasheet" "" (at 187.96 63.5 0)
+      (effects (font (size 1.27 1.27)) hide)
+    )
+    (property "MF" "Keystone Electronics Corp." (at 187.96 63.5 0)
+      (effects (font (size 1.27 1.27)) (justify bottom) hide)
+    )
+    (property "MAXIMUM_PACKAGE_HEIGHT" "4.57 mm" (at 187.96 63.5 0)
+      (effects (font (size 1.27 1.27)) (justify bottom) hide)
+    )
+    (property "Package" "None" (at 187.96 63.5 0)
+      (effects (font (size 1.27 1.27)) (justify bottom) hide)
+    )
+    (property "Price" "None" (at 187.96 63.5 0)
+      (effects (font (size 1.27 1.27)) (justify bottom) hide)
+    )
+    (property "Check_prices" "https://www.snapeda.com/parts/5001/Keystone+Electronics/view-part/?ref=eda" (at 187.96 63.5 0)
+      (effects (font (size 1.27 1.27)) (justify bottom) hide)
+    )
+    (property "STANDARD" "Manufacturer Recommendations" (at 187.96 63.5 0)
+      (effects (font (size 1.27 1.27)) (justify bottom) hide)
+    )
+    (property "PARTREV" "H" (at 187.96 63.5 0)
+      (effects (font (size 1.27 1.27)) (justify bottom) hide)
+    )
+    (property "SnapEDA_Link" "https://www.snapeda.com/parts/5001/Keystone+Electronics/view-part/?ref=snap" (at 187.96 63.5 0)
+      (effects (font (size 1.27 1.27)) (justify bottom) hide)
+    )
+    (property "MP" "5001" (at 187.96 63.5 0)
+      (effects (font (size 1.27 1.27)) (justify bottom) hide)
+    )
+    (property "Description" "\nBlack PC Test Point, Miniature Phosphor Bronze Silver Plating 0.040 (1.02mm) Hole Diameter Mounting Type\n" (at 187.96 63.5 0)
+      (effects (font (size 1.27 1.27)) (justify bottom) hide)
+    )
+    (property "MANUFACTURER" "Keystone" (at 187.96 63.5 0)
+      (effects (font (size 1.27 1.27)) (justify bottom) hide)
+    )
+    (property "Availability" "In Stock" (at 187.96 63.5 0)
+      (effects (font (size 1.27 1.27)) (justify bottom) hide)
+    )
+    (property "SNAPEDA_PN" "5000" (at 187.96 63.5 0)
+      (effects (font (size 1.27 1.27)) (justify bottom) hide)
+    )
+    (pin "TP")
+    (instances
+      (project "SiC based Battery Disconnect"
+        (path "/525387b1-1528-4728-a616-6f57d2a34d69/a4af0f90-9694-45a8-86a1-2f9082dd6b02"
+          (reference "TP9") (unit 1)
+        )
+        (path "/525387b1-1528-4728-a616-6f57d2a34d69/b74c6b34-d7cd-41a9-8566-5a1ea50c5493"
+          (reference "TP7") (unit 1)
+        )
+      )
+    )
+  )
   (symbol (lib_id "power:GND") (at 134.62 134.62 0) (unit 1)
     (in_bom yes) (on_board yes) (dnp no) (fields_autoplaced)
@@
         )
       )
+    )
+  )
+  (symbol (lib_id "5001:5001") (at 191.77 100.33 90) (unit 1)
+    (in_bom yes) (on_board yes) (dnp no) (fields_autoplaced)
+    (property "Reference" "TP9" (at 194.31 99.06 90)
+      (effects (font (size 1.27 1.27)) (justify right))
+    )
+    (property "Value" "5001" (at 194.31 101.6 90)
+      (effects (font (size 1.27 1.27)) (justify right))
+    )
+    (property "Footprint" "5001 tp:KEYSTONE_5001" (at 191.77 100.33 0)
+      (effects (font (size 1.27 1.27)) (justify bottom) hide)
+    )
+    (property "Datasheet" "" (at 191.77 100.33 0)
+      (effects (font (size 1.27 1.27)) hide)
+    )
+    (property "MF" "Keystone Electronics Corp." (at 191.77 100.33 0)
+      (effects (font (size 1.27 1.27)) (justify bottom) hide)
+    )
+    (property "MAXIMUM_PACKAGE_HEIGHT" "4.57 mm" (at 191.77 100.33 0)
+      (effects (font (size 1.27 1.27)) (justify bottom) hide)
+    )
+    (property "Package" "None" (at 191.77 100.33 0)
+      (effects (font (size 1.27 1.27)) (justify bottom) hide)
+    )
+    (property "Price" "None" (at 191.77 100.33 0)
+      (effects (font (size 1.27 1.27)) (justify bottom) hide)
+    )
+    (property "Check_prices" "https://www.snapeda.com/parts/5001/Keystone+Electronics/view-part/?ref=eda" (at 191.77 100.33 0)
+      (effects (font (size 1.27 1.27)) (justify bottom) hide)
+    )
+    (property "STANDARD" "Manufacturer Recommendations" (at 191.77 100.33 0)
+      (effects (font (size 1.27 1.27)) (justify bottom) hide)
+    )
+    (property "PARTREV" "H" (at 191.77 100.33 0)
+      (effects (font (size 1.27 1.27)) (justify bottom) hide)
+    )
+    (property "SnapEDA_Link" "https://www.snapeda.com/parts/5001/Keystone+Electronics/view-part/?ref=snap" (at 191.77 100.33 0)
+      (effects (font (size 1.27 1.27)) (justify bottom) hide)
+    )
+    (property "MP" "5001" (at 191.77 100.33 0)
+      (effects (font (size 1.27 1.27)) (justify bottom) hide)
+    )
+    (property "Description" "\nBlack PC Test Point, Miniature Phosphor Bronze Silver Plating 0.040 (1.02mm) Hole Diameter Mounting Type\n" (at 191.77 100.33 0)
+      (effects (font (size 1.27 1.27)) (justify bottom) hide)
+    )
+    (property "MANUFACTURER" "Keystone" (at 191.77 100.33 0)
+      (effects (font (size 1.27 1.27)) (justify bottom) hide)
+    )
+    (property "Availability" "In Stock" (at 191.77 100.33 0)
+      (effects (font (size 1.27 1.27)) (justify bottom) hide)
+    )
+    (property "SNAPEDA_PN" "5000" (at 191.77 100.33 0)
+      (effects (font (size 1.27 1.27)) (justify bottom) hide)
+    )
+    (pin "TP")
+    (instances
+      (project "SiC based Battery Disconnect"
+        (path "/525387b1-1528-4728-a616-6f57d2a34d69/a4af0f90-9694-45a8-86a1-2f9082dd6b02"
+          (reference "TP9") (unit 1)
+        )
+        (path "/525387b1-1528-4728-a616-6f57d2a34d69/b74c6b34-d7cd-41a9-8566-5a1ea50c5493"
+          (reference "TP6") (unit 1)
+        )
+      )

Commit message: Design with footprint error
Parts:
- U2: footprint Package_SO:TSSOP-8_4.4x3mm_P0.65mm -> MCP6022-E_SN:SOIC127P599X175-8N
Changed lines of the file:
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@@
       (effects (font (size 1.27 1.27)) (justify left))
     )
-    (property "Footprint" "Package_SO:TSSOP-8_4.4x3mm_P0.65mm" (at 154.94 110.49 0)
+    (property "Footprint" "MCP6022-E_SN:SOIC127P599X175-8N" (at 154.94 110.49 0)
       (effects (font (size 1.27 1.27)) hide)
     )
@@
       (effects (font (size 1.27 1.27)))
     )
-    (property "Footprint" "Package_SO:TSSOP-8_4.4x3mm_P0.65mm" (at 154.94 110.49 0)
+    (property "Footprint" "MCP6022-E_SN:SOIC127P599X175-8N" (at 154.94 110.49 0)
       (effects (font (size 1.27 1.27)) hide)
     )
@@
       (effects (font (size 1.27 1.27)))
     )
-    (property "Footprint" "Package_SO:TSSOP-8_4.4x3mm_P0.65mm" (at 147.32 73.66 0)
-      (effects (font (size 1.27 1.27)) hide)
-    )
+    (property "Footprint" "MCP6022-E_SN:SOIC127P599X175-8N" (at 147.32 73.66 0)
+      (effects (font (size 1.27 1.27)) hide)
+    )

Commit message: Final Design
Parts:
- added C6: 0.1uF, Capacitor_SMD:C_0805_2012Metric, symbol Device:C
Connections:
- net GND: now also C6.2
- net VDDHV: now also C6.1
Other:
- moved on the sheet: C10, R12, TP9, U2A, U2C
